File: kicad/chonky/chonky.kicad_pcb (KiCad board)
At the start: 2 copper layers, 35 parts, among them SW00 SW_Push, SW01 SW_Push, SW02 SW_Push, SW03 SW_Push, SW04 SW_Push, SW10 SW_Push, SW11 SW_Push, SW12 SW_Push, SW13 SW_Push, SW14 SW_Push, SW20 SW_Push, SW21 SW_Push, SW22 SW_Push, SW23 SW_Push, SW24 SW_Push, SW33 SW_Push, SW34 SW_Push, U1 ProMicro

Commit message: Too lazy to comment
Parts:
- D00, D01, D02, D03, D04, D10, D11, D12, D13, D14, D20, D21, D22, D23, D24, D33, D34: footprint Diode_THT:D_DO-35_SOD27_P7.62mm_Horizontal -> Diode_SMD:D_SOD-123
- moved D10 176.3 mm to (-117.8, 69.0), turned to 1 degrees
- moved D20 175.4 mm to (-117.4, 92.1), turned to 1 degrees
- moved D00 170.1 mm to (-112.7, 56.3), turned to 91 degrees
- moved SW00 166.3 mm to (-122.3, 51.6), turned to -179 degrees
- moved SW10 165.7 mm to (-121.9, 74.6), turned to -179 degrees
- moved SW20 165.1 mm to (-121.6, 97.6), turned to -179 degrees
